Commit message: Added imu to urdf and for gazebo simulation

File: src/bumperbot_description/urdf/bumperbot.urdf.xacro (robot description, xacro)
@@ -138,4 +138,31 @@
         <child link="caster_rear_link"/>
     </joint>
+    <link name="imu_link">
+        <inertial>
+            <origin xyz="-0.00552433659106688 0.000168210391520346 0.000514000497342681" rpy="0 0 0" />
+            <mass value="0.000528415362211671" />
+            <inertia ixx="1.46176048428261E-08" ixy="1.40015117949421E-10" ixz="-1.99633872937403E-12"
+                iyy="8.59662482954888E-09" iyz="7.52375112767959E-12"
+                izz="2.30279421279312E-08" />
+            </inertial>
+        <visual>
+            <origin xyz="0 0 0" rpy="0 0 0" />
+            <geometry>
+                <mesh filename="package://bumperbot_description/meshes/imu_link.STL" />
+            </geometry>
+        </visual>
+        <collision>
+            <origin xyz="0 0 0" rpy="0 0 0" />
+            <geometry>
+                <mesh filename="package://bumperbot_description/meshes/imu_link.STL" />
+            </geometry>
+        </collision>
+    </link>
+    <joint name="imu_joint" type="fixed">
+        <origin xyz="0 0 0.07" rpy="3.14 0 0"/>
+        <parent link="base_link"/>
+        <child link="imu_link"/>
+        <axis xyz="0 0 0" />
+    </joint>
     <!-- Insert Can
     <link name="can_link">

File: src/bumperbot_description/urdf/bumperbot_gazebo.xacro (robot description, xacro)
@@ -67,3 +67,14 @@
         </plugin>
     </gazebo>
+    <gazebo>
+      <plugin name="imu_plugin" filename="libgazebo_ros_imu.so">
+        <alwaysOn>true</alwaysOn>
+        <bodyName>imu_link</bodyName>
+        <frameName>imu_link</frameName>
+        <topicName>imu</topicName>
+        <serviceName>imu_service</serviceName>
+        <gaussianNoise>0.001</gaussianNoise>
+        <updateRate>1000</updateRate>
+      </plugin>
+    </gazebo>
 </robot>

Commit message: Added sensor fusion functionality using localization package

File: src/bumperbot_description/urdf/bumperbot.urdf.xacro (robot description, xacro)
@@ -160,7 +160,7 @@
     </link>
     <joint name="imu_joint" type="fixed">
-        <origin xyz="0 0 0.07" rpy="3.14 0 0"/>
-        <parent link="base_link"/>
-        <child link="imu_link"/>
+        <origin xyz="0 0 0.0698986241758014" rpy="3.14159265358979 0 0" />
+        <parent link="base_link" />
+        <child link="imu_link" />
         <axis xyz="0 0 0" />
     </joint>

Commit message: Initial Push

File: src/bumperbot_description/urdf/bumperbot.urdf.xacro (robot description, xacro)
@@ -165,12 +165,37 @@
         <axis xyz="0 0 0" />
     </joint>
-    <!-- Insert Can
-    <link name="can_link">
-    <visual>
-        <origin xyz="0.03 0.03 0" rpy="1.57 0 0"/>
-        <geometry>
-            <mesh filename="package://bumperbot_description/meshes/can.STL" />
-        </geometry>
-    </visual>
+    <link name="lidar_1_link">
+        <collision>
+            <origin xyz="0 0 0" rpy="0 0 0"/>
+            <geometry>
+          <box size="0.01 0.01 0.01"/>
+            </geometry>
+          </collision>
+          <visual>
+            <origin xyz="0 0 0" rpy="0 0 0"/>
+            <geometry>
+                <cylinder radius="0.01" length="0.01"/>
+            </geometry>
+          </visual>
+          <inertial>
+            <mass value="1e-5" />
+            <origin xyz="0 0 0" rpy="0 0 0"/>
+            <inertia ixx="1e-6" ixy="0" ixz="0" iyy="1e-6" iyz="0" izz="1e-6" />
+          </inertial>
+    </link>
+    <joint name="lidar_1_joint" type="fixed">
+        <axis xyz="0 1 0" />
+        <origin xyz="0.0 0.0 0.08" rpy="0 0 0"/>
+        <parent link="base_link"/>
+        <child link="lidar_1_link"/>
+    </joint>
+    <!-- Insert Can -->
+    <!-- <link name="can_link">
+        <visual>
+            <origin xyz="0.03 0.03 0" rpy="1.57 0 0"/>
+            <geometry>
+                <mesh filename="package://bumperbot_description/meshes/can.STL" />
+            </geometry>
+        </visual>
     </link>
     <joint name="can_joint" type="fixed">

File: src/bumperbot_description/urdf/bumperbot_gazebo.xacro (robot description, xacro)
@@ -78,3 +78,39 @@
       </plugin>
     </gazebo>
+     <!-- Lidar 1 -->
+    <gazebo reference="lidar_1_link">
+      <sensor type="ray" name="head_hokuyo_sensor">
+        <pose>0 0 0 0 0 0</pose>
+        <visualize>true</visualize>
+        <update_rate>20</update_rate>
+        <ray>
+          <scan>
+            <horizontal>
+              <samples>720</samples>
+              <resolution>1</resolution>
+              <min_angle>-3.14</min_angle>
+              <max_angle>3.14</max_angle>
+            </horizontal>
+          </scan>
+          <range>
+            <min>0.3</min>
+            <max>20.0</max>
+            <resolution>0.01</resolution>
+          </range>
+          <noise>
+            <type>gaussian</type>
+            <!-- Noise parameters based on published spec for Hokuyo laser
+                achieving "+-30mm" accuracy at range < 10m.  A mean of 0.0m and
+                stddev of 0.01m will put 99.7% of samples within 0.03m of the true
+                reading. -->
+            <mean>0.0</mean>
+            <stddev>0.01</stddev>
+          </noise>
+        </ray>
+        <plugin name="gazebo_ros_head_hokuyo_controller" filename="libgazebo_ros_laser.so">
+          <topicName>/bumperbot/laser/scan</topicName>
+          <frameName>lidar_1_link</frameName>
+        </plugin>
+      </sensor>
+    </gazebo>
 </robot>

Commit message: Added depth camera and lidar

File: src/bumperbot_description/urdf/bumperbot.urdf.xacro (robot description, xacro)
@@ -165,29 +165,8 @@
         <axis xyz="0 0 0" />
     </joint>
-    <link name="lidar_1_link">
-        <collision>
-            <origin xyz="0 0 0" rpy="0 0 0"/>
-            <geometry>
-          <box size="0.01 0.01 0.01"/>
-            </geometry>
-          </collision>
-          <visual>
-            <origin xyz="0 0 0" rpy="0 0 0"/>
-            <geometry>
-                <cylinder radius="0.01" length="0.01"/>
-            </geometry>
-          </visual>
-          <inertial>
-            <mass value="1e-5" />
-            <origin xyz="0 0 0" rpy="0 0 0"/>
-            <inertia ixx="1e-6" ixy="0" ixz="0" iyy="1e-6" iyz="0" izz="1e-6" />
-          </inertial>
-    </link>
-    <joint name="lidar_1_joint" type="fixed">
-        <axis xyz="0 1 0" />
-        <origin xyz="0.0 0.0 0.08" rpy="0 0 0"/>
-        <parent link="base_link"/>
-        <child link="lidar_1_link"/>
-    </joint>
+    <!-- Lidar -->
+    <xacro:include filename="lidar.xacro" />
+    <!-- Depth Camera (RGBD) -->
+    <xacro:include filename="depth_camera.xacro" />
     <!-- Insert Can -->
     <!-- <link name="can_link">

File: src/bumperbot_description/urdf/bumperbot_gazebo.xacro (robot description, xacro)
@@ -78,39 +78,3 @@
       </plugin>
     </gazebo>
-     <!-- Lidar 1 -->
-    <gazebo reference="lidar_1_link">
-      <sensor type="ray" name="head_hokuyo_sensor">
-        <pose>0 0 0 0 0 0</pose>
-        <visualize>true</visualize>
-        <update_rate>20</update_rate>
-        <ray>
-          <scan>
-            <horizontal>
-              <samples>720</samples>
-              <resolution>1</resolution>
-              <min_angle>-3.14</min_angle>
-              <max_angle>3.14</max_angle>
-            </horizontal>
-          </scan>
-          <range>
-            <min>0.3</min>
-            <max>20.0</max>
-            <resolution>0.01</resolution>
-          </range>
-          <noise>
-            <type>gaussian</type>
-            <!-- Noise parameters based on published spec for Hokuyo laser
-                achieving "+-30mm" accuracy at range < 10m.  A mean of 0.0m and
-                stddev of 0.01m will put 99.7% of samples within 0.03m of the true
-                reading. -->
-            <mean>0.0</mean>
-            <stddev>0.01</stddev>
-          </noise>
-        </ray>
-        <plugin name="gazebo_ros_head_hokuyo_controller" filename="libgazebo_ros_laser.so">
-          <topicName>/bumperbot/laser/scan</topicName>
-          <frameName>lidar_1_link</frameName>
-        </plugin>
-      </sensor>
-    </gazebo>
 </robot>
