Commit message: added robot params into config file

File: src/bumperbot_description/urdf/2d_lidar.xacro (robot description, xacro)
@@ -1,4 +1,8 @@
 <?xml version="1.0"?>
 <robot name="bumperbot" xmlns:xacro="http://ros.org/wiki/xacro">
+     <!-- Load robot params file -->
+    <xacro:property name="robot_params_file" value="$(find config_manager)/config/robot_config.yaml"/>
+    <xacro:property name="robot_params" value="${xacro.load_yaml(robot_params_file)}"/>
+    <xacro:property name="lidar_params_2d" value="${robot_params['lidar_2d']}"/>
     <!-- Left LIDAR -->
     <link name="lidar_left_link">
@@ -58,27 +62,27 @@
         <pose>0 0 0 0 0 0</pose>
         <visualize>true</visualize>
-        <update_rate>20</update_rate>
+        <update_rate>${lidar_params_2d['left']['update_rate']}</update_rate>
         <ray>
             <scan>
             <horizontal>
-                <samples>720</samples>
-                <resolution>1</resolution>
-                <min_angle>${-pi/2}</min_angle>
-                <max_angle>${pi/2}</max_angle>
+                <samples>${lidar_params_2d['left']['horizontal_scan']['sample']}</samples>
+                <resolution>${lidar_params_2d['left']['horizontal_scan']['resolution']}</resolution>
+                <min_angle>${lidar_params_2d['left']['horizontal_scan']['min_angle']}</min_angle>
+                <max_angle>${lidar_params_2d['left']['horizontal_scan']['max_angle']}</max_angle>
             </horizontal>
             </scan>
             <range>
-            <min>0.3</min>
-            <max>20.0</max>
-            <resolution>0.01</resolution>
+                <min>${lidar_params_2d['left']['range']['min']}</min>
+                <max>${lidar_params_2d['left']['range']['max']}</max>
+                <resolution>${lidar_params_2d['left']['range']['resolution']}</resolution>
             </range>
             <noise>
-            <type>gaussian</type>
-            <!-- Noise parameters based on published spec for Hokuyo laser
-                achieving "+-30mm" accuracy at range < 10m.  A mean of 0.0m and
-                stddev of 0.01m will put 99.7% of samples within 0.03m of the true
-                reading. -->
-            <mean>0.0</mean>
-            <stddev>0.01</stddev>
+                <type>gaussian</type>
+                <!-- Noise parameters based on published spec for Hokuyo laser
+                    achieving "+-30mm" accuracy at range < 10m.  A mean of 0.0m and
+                    stddev of 0.01m will put 99.7% of samples within 0.03m of the true
+                    reading. -->
+                <mean>${lidar_params_2d['left']['noise']['mean']}</mean>
+                <stddev>${lidar_params_2d['left']['noise']['stddev']}</stddev>
             </noise>
         </ray>
@@ -94,27 +98,27 @@
         <pose>0 0 0 0 0 0</pose>
         <visualize>true</visualize>
-        <update_rate>20</update_rate>
+        <update_rate>${lidar_params_2d['right']['update_rate']}</update_rate>
         <ray>
             <scan>
             <horizontal>
-                <samples>720</samples>
-                <resolution>1</resolution>
-                <min_angle>${-pi/2}</min_angle>
-                <max_angle>${pi/2}</max_angle>
+                <samples>${lidar_params_2d['right']['horizontal_scan']['sample']}</samples>
+                <resolution>${lidar_params_2d['right']['horizontal_scan']['resolution']}</resolution>
+                <min_angle>${lidar_params_2d['right']['horizontal_scan']['min_angle']}</min_angle>
+                <max_angle>${lidar_params_2d['right']['horizontal_scan']['max_angle']}</max_angle>
             </horizontal>
             </scan>
             <range>
-            <min>0.3</min>
-            <max>20.0</max>
-            <resolution>0.01</resolution>
+                <min>${lidar_params_2d['right']['range']['min']}</min>
+                <max>${lidar_params_2d['right']['range']['max']}</max>
+                <resolution>${lidar_params_2d['right']['range']['resolution']}</resolution>
             </range>
             <noise>
-            <type>gaussian</type>
-            <!-- Noise parameters based on published spec for Hokuyo laser
-                achieving "+-30mm" accuracy at range < 10m.  A mean of 0.0m and
-                stddev of 0.01m will put 99.7% of samples within 0.03m of the true
-                reading. -->
-            <mean>0.0</mean>
-            <stddev>0.01</stddev>
+                <type>gaussian</type>
+                <!-- Noise parameters based on published spec for Hokuyo laser
+                    achieving "+-30mm" accuracy at range < 10m.  A mean of 0.0m and
+                    stddev of 0.01m will put 99.7% of samples within 0.03m of the true
+                    reading. -->
+                <mean>${lidar_params_2d['right']['noise']['mean']}</mean>
+                <stddev>${lidar_params_2d['right']['noise']['stddev']}</stddev>
             </noise>
         </ray>

File: src/bumperbot_description/urdf/3d_velodyne_lidar.xacro (robot description, xacro)
@@ -1,4 +1,8 @@
 <?xml version="1.0"?>
 <robot name="bumperbot" xmlns:xacro="http://ros.org/wiki/xacro">
+    <!-- Load robot params file -->
+    <xacro:property name="robot_params_file" value="$(find config_manager)/config/robot_config.yaml"/>
+    <xacro:property name="robot_params" value="${xacro.load_yaml(robot_params_file)}"/>
+    <xacro:property name="lidar_params_3d" value="${robot_params['lidar_3d']}"/>
     <!-- Velodyne 3D Lidar -->
     <link name="velodyne_link">
@@ -32,29 +36,29 @@
             <pose>0 0 0 0 0 0</pose>
             <visualize>false</visualize>
-            <update_rate>20</update_rate>
+            <update_rate>${lidar_params_3d['update_rate']}</update_rate>
             <ray>
                 <scan>
                     <horizontal>
-                        <samples>1440</samples>
-                        <resolution>1</resolution>
-                        <min_angle>${-pi}</min_angle>  <!-- -180 degrees -->
-                        <max_angle>${pi}</max_angle>   <!-- 180 degrees -->
+                        <samples>${lidar_params_3d['horizontal_scan']['sample']}</samples>
+                        <resolution>${lidar_params_3d['horizontal_scan']['resolution']}</resolution>
+                        <min_angle>${lidar_params_3d['horizontal_scan']['min_angle']}</min_angle>  <!-- -180 degrees -->
+                        <max_angle>${lidar_params_3d['horizontal_scan']['max_angle']}</max_angle>   <!-- 180 degrees -->
                     </horizontal>
                     <vertical>
-                        <samples>16</samples>
-                        <resolution>1</resolution>
-                        <min_angle>0</min_angle>   <!-- Vertical min angle -->
-                        <max_angle>0.2618</max_angle>   <!-- Vertical max angle -->
+                        <samples>${lidar_params_3d['vertical_scan']['sample']}</samples>
+                        <resolution>${lidar_params_3d['vertical_scan']['resolution']}</resolution>
+                        <min_angle>${lidar_params_3d['vertical_scan']['min_angle']}</min_angle>   <!-- Vertical min angle -->
+                        <max_angle>${lidar_params_3d['vertical_scan']['max_angle']}</max_angle>   <!-- Vertical max angle -->
                     </vertical>
                 </scan>
                 <range>
-                    <min>0.1</min>
-                    <max>70.0</max>
-                    <resolution>0.001</resolution>
+                    <min>${lidar_params_3d['range']['min']}</min>
+                    <max>${lidar_params_3d['range']['max']}</max>
+                    <resolution>${lidar_params_3d['range']['resolution']}</resolution>
                 </range>
                 <noise>
                     <type>gaussian</type>
-                    <mean>0.0</mean>
-                    <stddev>0.01</stddev>
+                    <mean>${lidar_params_3d['noise']['mean']}</mean>
+                    <stddev>${lidar_params_3d['noise']['stddev']}</stddev>
                 </noise>
             </ray>

File: src/bumperbot_description/urdf/bumperbot.urdf.xacro (robot description, xacro)
@@ -3,4 +3,10 @@
     <!-- Include other xacro models into this file -->
     <xacro:include filename="$(find bumperbot_description)/urdf/bumperbot_gazebo.xacro"/>
+    <!-- Load robot params file -->
+    <xacro:property name="robot_params_file" value="$(find config_manager)/config/robot_config.yaml"/>
+    <xacro:property name="robot_params" value="${xacro.load_yaml(robot_params_file)}"/>
+    <xacro:property name="wheel_params" value="${robot_params['wheel']}"/>
+    <xacro:property name="caster_wheel_params" value="${robot_params['caster_wheel']}"/>
+    <xacro:property name="base_link_params" value="${robot_params['base_link']}"/>
     <!-- Parent link for all other links -->
     <!-- Also acts as interface between robot and surrounding env -->
@@ -49,10 +55,10 @@
             <origin xyz="0.0 -0.015 0.0" rpy="1.57 0.0 0.0"/>
             <geometry>
-                <sphere radius="0.033"/>
+                <sphere radius="${wheel_params['radius']}"/>
             </geometry>
         </collision>
     </link>
     <joint name="wheel_right_joint" type="continuous">
-        <origin rpy="0 0 0" xyz="0 -0.07 0" />
+        <origin rpy="0 0 0" xyz="0 -${wheel_params['separation']/2} 0" />
         <parent link="base_link"/>
         <child link="wheel_right_link"/>
@@ -76,10 +82,10 @@
             <origin xyz="0.0 0.015 0.0" rpy="1.57 0.0 0.0"/>
             <geometry>
-                <sphere radius="0.033"/>
+                <sphere radius="${wheel_params['radius']}"/>
             </geometry>
         </collision>
     </link>
     <joint name="wheel_left_joint" type="continuous">
-        <origin rpy="0 0 0" xyz="0 0.07 0" />
+        <origin rpy="0 0 0" xyz="0 ${wheel_params['separation']/2} 0" />
         <parent link="base_link"/>
         <child link="wheel_left_link"/>
@@ -103,5 +109,5 @@
             <origin xyz="0.0 0.0 0.0" rpy="0.0 0.0 0.0"/>
             <geometry>
-                <sphere radius="0.005"/>
+                <sphere radius="${caster_wheel_params['radius']}"/>
             </geometry>
         </collision>
@@ -129,5 +135,5 @@
             <origin xyz="0.0 0.0 0.0" rpy="0.0 0.0 0.0"/>
             <geometry>
-                <sphere radius="0.005"/>
+                <sphere radius="${caster_wheel_params['radius']}"/>
             </geometry>
         </collision>

File: src/bumperbot_description/urdf/depth_camera.xacro (robot description, xacro)
@@ -1,8 +1,12 @@
 <?xml version="1.0"?>
 <robot name="bumperbot" xmlns:xacro="http://ros.org/wiki/xacro">
+    <!-- Load robot params file -->
+    <xacro:property name="robot_params_file" value="$(find config_manager)/config/robot_config.yaml"/>
+    <xacro:property name="robot_params" value="${xacro.load_yaml(robot_params_file)}"/>
+    <xacro:property name="camera_params" value="${robot_params['litter_detection']}"/>
     <joint name="camera_joint" type="fixed">
         <parent link="base_link"/>
         <child link="dpcamera_link"/>
-        <origin xyz="0.072 0.0 0.065" rpy="0.0 0.2618 0.0"/>
+        <origin xyz="0.072 0.0 0.065" rpy="0.0 ${camera_params['camera_theta']} 0.0"/>
     </joint>
     <link name="dpcamera_link">
