Commit message: Create detection tf from camera frame to base footprint, fix detection coordinate

File: src/bumperbot_description/urdf/depth_camera.xacro (robot description, xacro)
@@ -4,5 +4,5 @@
         <parent link="base_link"/>
         <child link="dpcamera_link"/>
-        <origin xyz="0.072 0.0 0.065" />
+        <origin xyz="0.072 0.0 0.065" rpy="0.0 0.2618 0.0"/>
     </joint>
     <link name="dpcamera_link">
@@ -29,4 +29,5 @@
             <camera>
                 <horizontal_fov>1.089</horizontal_fov>
+                <vertical_fov>1.089</vertical_fov>
                 <image>
                     <format>B8G8R8</format>
@@ -52,5 +53,5 @@
                 <pointCloudTopicName>/camera/depth/points</pointCloudTopicName>
                 <frameName>dpcamera_link</frameName>
-                <pointCloudCutoff>0.5</pointCloudCutoff>
+                <pointCloudCutoff>0.05</pointCloudCutoff>
                 <pointCloudCutoffMax>3.0</pointCloudCutoffMax>
                 <distortionK1>0</distortionK1>

Commit message: fix compressedImage topic, added topic and transformations for rear camera, changed transformation target to base_link

File: src/bumperbot_description/urdf/depth_camera.xacro (robot description, xacro)
@@ -51,9 +51,9 @@
                 <updateRate>0.0</updateRate>
                 <cameraName>camera_ir</cameraName>
-                <imageTopicName>/depth_camera/color/image_raw</imageTopicName>
-                <cameraInfoTopicName>/depth_camera/color/camera_info</cameraInfoTopicName>
-                <depthImageTopicName>/depth_camera/depth/image_raw</depthImageTopicName>
-                <depthImageCameraInfoTopicName>/depth_camera/depth/camera_info</depthImageCameraInfoTopicName>
-                <pointCloudTopicName>/depth_camera/depth/points</pointCloudTopicName>
+                <imageTopicName>/depth_camera_front/color/image_raw</imageTopicName>
+                <cameraInfoTopicName>/depth_camera_front/color/camera_info</cameraInfoTopicName>
+                <depthImageTopicName>/depth_camera_front/depth/image_raw</depthImageTopicName>
+                <depthImageCameraInfoTopicName>/depth_camera_front/depth/camera_info</depthImageCameraInfoTopicName>
+                <pointCloudTopicName>/depth_camera_front/depth/points</pointCloudTopicName>
                 <frameName>dpcamera_link</frameName>
                 <pointCloudCutoff>0.05</pointCloudCutoff>
@@ -77,3 +77,70 @@
         </sensor>
     </gazebo>
+    <joint name="rear_camera_joint" type="fixed">
+        <parent link="base_link"/>
+        <child link="rear_dpcamera_link"/>
+        <origin xyz="-0.072 0.0 0.065" rpy="0.0 ${camera_params['camera_theta']} ${pi}"/>
+    </joint>
+    <link name="rear_dpcamera_link">
+        <visual>
+            <geometry>
+                <box size="0.010 0.03 0.03"/>
+            </geometry>
+            <material name="blue"/>
+        </visual>
+    </link>
+    <joint name="rear_camera_optical_joint" type="fixed">
+        <parent link="rear_dpcamera_link"/>
+        <child link="rear_dpcamera_link_optical"/>
+        <origin xyz="0.0 0.0 0.0" rpy="0.0 ${-pi/2} 0.0"/>
+    </joint>
+    <link name="rear_dpcamera_link_optical" />
+    <!-- Gazebo: rear_dpcamera_link -->
+    <gazebo reference="rear_dpcamera_link">
+        <material>Gazebo/Blue</material>
+        <sensor name="rear_camera" type="depth">
+            <pose> 0 0 0 0 0 0 </pose>
+            <visualize>true</visualize>
+            <update_rate>10</update_rate>
+            <camera>
+                <horizontal_fov>1.089</horizontal_fov>
+                <vertical_fov>1.089</vertical_fov>
+                <image>
+                    <format>B8G8R8</format>
+                    <width>640</width>
+                    <height>480</height>
+                </image>
+                <clip>
+                    <near>0.05</near>
+                    <far>8.0</far>
+                </clip>
+            </camera>
+            <plugin name="camera_plugin" filename="libgazebo_ros_openni_kinect.so">
+                <baseline>0.2</baseline>
+                <alwaysOn>true</alwaysOn>
+                <!-- Keep this zero, update_rate in the parent <sensor> tag
+                    will control the frame rate. -->
+                <updateRate>0.0</updateRate>
+                <cameraName>rear_camera_ir</cameraName>
+                <imageTopicName>/depth_camera_rear/color/image_raw</imageTopicName>
+                <cameraInfoTopicName>/depth_camera_rear/color/camera_info</cameraInfoTopicName>
+                <depthImageTopicName>/depth_camera_rear/depth/image_raw</depthImageTopicName>
+                <depthImageCameraInfoTopicName>/depth_camera_rear/depth/camera_info</depthImageCameraInfoTopicName>
+                <pointCloudTopicName>/depth_camera_rear/depth/points</pointCloudTopicName>
+                <frameName>rear_dpcamera_link</frameName>
+                <pointCloudCutoff>0.05</pointCloudCutoff>
+                <pointCloudCutoffMax>3.0</pointCloudCutoffMax>
+                <distortionK1>0</distortionK1>
+                <distortionK2>0</distortionK2>
+                <distortionK3>0</distortionK3>
+                <distortionT1>0</distortionT1>
+                <distortionT2>0</distortionT2>
+                <CxPrime>0</CxPrime>
+                <Cx>0</Cx>
+                <Cy>0</Cy>
+                <focalLength>0</focalLength>
+                <hackBaseline>0</hackBaseline>
+            </plugin>
+        </sensor>
+    </gazebo>
 </robot>
